File: hardware/XYZ_adapter_v2/schematic_rxtx_adapter.brd (EAGLE design)
At the start: 160 x 100 mm, 18 parts, among them Q1 2N7002E, Q2 2N7002E

Commit message: Updated xyz_adapter_v2
Parts:
- removed GND, GND2, GND3, GND4, PAD3, PAD4, RX_IN, RX_OUT, TX_IN, TX_OUT, VDD: (no value), wirepad:1,6/0,8
- added SV1: (no value), con-lstb:MA06-1
- moved Q1 2.29 mm to (27.7, 41.9)
- moved R2 1.61 mm to (31.5, 30.5), turned to 270 degrees
- moved R3 1.55 mm to (22.1, 29.2), turned to 270 degrees
- moved R1 1.44 mm to (17.3, 30.5), turned to 270 degrees
- moved R4 1.05 mm to (26.9, 29.2), turned to 270 degrees
- flipped X1 to the bottom
Connections:
- removed net N$1: Q1.2, R1.1, TX_IN.1
- removed net N$2: PAD4.1, R2.2, R4.2
- removed net N$3: Q1.3, R2.1, TX_OUT.1, X1.3
- removed net N$5: Q2.2, R3.1, RX_IN.1
- removed net N$6: PAD3.1, Q1.1, Q2.1, R1.2, R3.2
- removed net N$7: VDD.1, X1.2
- removed net N$8: Q2.3, R4.1, RX_OUT.1, X1.4
- new net RX_IN: Q2.2, R3.1, SV1.3
- new net RX_OUT: Q2.3, R4.1, X1.4
- new net TX_IN: Q1.2, R1.1, SV1.2
- new net TX_OUT: Q1.3, R2.1, X1.3
- new net VDD: SV1.4, X1.2
- new net VREF: Q1.1, Q2.1, R1.2, R2.2, R3.2, R4.2, SV1.1
- net GND: now also SV1.5, SV1.6; no longer GND.1, GND2.1, GND3.1, GND4.1
Routing:
- net VREF: track 0.00 -> 71.9 mm, vias 0 -> 3
- net N$3: track 69.4 -> 0.00 mm, vias 5 -> 0
- net N$5: track 57.3 -> 0.00 mm
- net N$8: track 54.6 -> 0.00 mm
- net GND: track 71.9 -> 22.0 mm
- net N$1: track 35.4 -> 0.00 mm
- net TX_IN: track 0.00 -> 34.9 mm
- net N$7: track 31.2 -> 0.00 mm, vias 2 -> 0
- net TX_OUT: track 0.00 -> 29.2 mm
- net N$6: track 24.6 -> 0.00 mm
- net RX_OUT: track 0.00 -> 24.3 mm
- net N$2: track 23.8 -> 0.00 mm, vias 2 -> 0
- net RX_IN: track 0.00 -> 20.4 mm
- net VDD: track 0.00 -> 18.7 mm
Other:
- board text added: "RX-TX XYZRobot v2"
- board text removed: "RX-TX XYZRobot v1"
