File: hardware/XYZ_adapter_v2/schematic_rxtx_adapter.sch (EAGLE design)
At the start: 18 parts, among them Q1 2N7002E, Q2 2N7002E

Commit message: Updated xyz_adapter_v2
Parts:
- removed GND, GND2, GND3, GND4, PAD3, PAD4, RX_IN, RX_OUT, TX_IN, TX_OUT, VDD: (no value), wirepad:1,6/0,8
- added SV1: (no value), con-lstb:MA06-1
Connections:
- removed net N$1: Q1.S, R1.1, TX_IN.P
- removed net N$2: PAD4.P, R2.2, R4.2
- removed net N$3: Q1.D, R2.1, TX_OUT.P, X1-3.S
- removed net N$5: Q2.S, R3.1, RX_IN.P
- removed net N$6: PAD3.P, Q1.G, Q2.G, R1.2, R3.2
- removed net N$7: VDD.P, X1-2.S
- removed net N$8: Q2.D, R4.1, RX_OUT.P, X1-4.S
- new net RX_IN: Q2.S, R3.1, SV1.3
- new net RX_OUT: Q2.D, R4.1, X1-4.S
- new net TX_IN: Q1.S, R1.1, SV1.2
- new net TX_OUT: Q1.D, R2.1, X1-3.S
- new net VDD: SV1.4, X1-2.S
- new net VREF: Q1.G, Q2.G, R1.2, R2.2, R3.2, R4.2, SV1.1
- net GND: now also SV1.5, SV1.6; no longer GND.P, GND2.P, GND3.P, GND4.P
Other:
- note added: "GND"
- note added: "RX_IN"
- note added: "RX_OUT"
- note added: "TX_IN"
- note added: "TX_OUT"
- note added: "VDD"
- note added: "VREF"
